File: hardware/signal-generator/signal-generator.sch (KiCad schematic (older format))
At the start: 0 parts

Commit message: [Signal Generator] Draw power supply section of schematic
The board requires an external power supply which provides the following
power supply rails:
- +12VA/-12VA to AGND: for analog circuitry
- +5VD to DGND: for digital circuitry
The power supply is connected to the board via a 2x5 pin connector. The
received power supply rails are additionally smoothed out via some 10uF
capacitors.
Additionally, the board itself contains LDO voltage regulators to
produce two additional analog voltage rails: +5VA/-5VA (to AGND).
Parts:
- added C? (x3): 10uF/16V, symbol Device:CP
- added C? (x4): 2.2uF, symbol Device:C
- added J?: Power_Supply_Rails, symbol Connector_Generic:Conn_02x05_Odd_Even
- added U?: ADP7142AUZJ-5.0, Package_TO_SOT_SMD:TSOT-23-5, symbol Regulator_Linear:ADP7142AUZJ
- added U?: ADP7182AUZJ-5.0, Package_TO_SOT_SMD:TSOT-23-5, symbol Regulator_Linear:ADP7182AUZJ
Connections:
- net labels added: +12VA, +5VA, +5VD, -12VA, -5VA, AGND, DGND, GNDA, GNDD
- wire segments 0 -> 60
- no-connect marks 0 -> 3
Other:
- note added: "+5VA/-5VA RAILS"
- note added: "POWER FLAGS"
- note added: "POWER SUPPLY"
- note added: "SMOOTHING CAPACITORS"

Commit message: [Signal Generator] Design the DDS system
The project's Direct Digital Synthesis (DDS) system is responsible for
generating the various user-programmable waveforms, as well as setting
the generated signal's frequency. The whole system is encapsulated
within a KiCAD hierarchical sheet. More details on the working operation
of the DDS system may be found in the (future) documentation of this
project...soonTM
Connections:
- wire segments 60 -> 62
Changed lines of the file:
@@
 Sheet 1 3
 Title "Digital Function Generator v2"
-Date "2019-10-31"
+Date "2019-11-05"
 Rev "1"
 Comp "Petar Nikolov"
@@
 $EndDescr
 $Sheet
-S 4750 3300 1350 800
+S 4750 3300 1300 1100
 U 5DB72CF6
 F0 "DDS System" 50
 F1 "DDS-system.sch" 50
+F2 "IOUTA" I R 6050 3800 50
+F3 "IOUTB" I R 6050 3900 50
+F4 "~IOExRESET" I L 4750 3800 50
+F5 "R\\~W" I L 4750 4000 50
+F6 "~CMR1" I L 4750 3600 50
+F7 "~CMR2" I L 4750 3700 50
+F8 "SDA" I R 6050 3500 50
+F9 "SCL" I R 6050 3400 50
+F10 "PWRDWN" I L 4750 3400 50
+F11 "~OSCOE" I L 4750 4300 50
+F12 "~CP" I L 4750 4100 50
 $EndSheet
 $Comp
@@
 	4750 7100 4850 7100
 Wire Wire Line
-	4550 6300 4850 6500
-Wire Wire Line
-	5650 6500 5950 6300
+	4550 6300 4750 6500
+Wire Wire Line
+	5750 6500 5950 6300
 $Comp
 L power:GNDA #PWR0115
@@
 Text Notes 550  5200 0    50   ~ 0
 POWER SUPPLY
+Wire Wire Line
+	4850 6500 4750 6500
+Wire Wire Line
+	5750 6500 5650 6500
 $EndSCHEMATC
