File: hardware/signal-generator/output-circuitry.sch (KiCad schematic (older format))
At the start: 28 parts

Commit message: [Signal Generator] Add DAC output conversion stage
The additional opamp stage is a differential amplifier configuration
which converts the differential current outputs of the DAC to a singular
voltage output in the range -0.5V to +0.5V.

The electrical schematic has overall been finalized with this addition.
Parts:
- removed C?: 100nF, symbol Device:C
- removed R?: 2k, symbol Device:R
- removed U?: LM4040CYM3-2.5-TR, Package_TO_SOT_SMD:SOT-23, symbol Reference_Voltage:LM4040DBZ-2.5
- added C?: 6.8pF, symbol Device:C
- added C? (x3): 100nF, symbol Device:C
- added C?: 2.2nF, symbol Device:C
- added R? (x5): 1k, symbol Device:R
- added R?: 1k2, symbol Device:R
- added R? (x2): 15R, symbol Device:R
- added R? (x2): 10R, symbol Device:R
- added U?: AD8021ARZ, symbol ulib_IC_Amplifiers:AD8021ARZ
- added U?: LM4040CYM3-2.5-TR, Package_TO_SOT_SMD:SOT-23, symbol Reference_Voltage:LM4040DBZ-2.5
Connections:
- net labels added: INA, INB, VINamp
- net labels removed: VIN
- wire segments 157 -> 203
Other:
- note added: "DIFFERENTIAL AMPLIFIER"
- note added: "OFFSET REMOVAL AND TWO-TIMES AMPLIFICATION"
- note added: "WAVEFORM AMPLIFICATION"
- note added: "WAVEFORM DC OFFSET"
- moved on the sheet: C?, R?, U?

Commit message: [Signal Generator] Implement +3.3VD line with TC1017 voltage regulator
Up until now, the +3.3VD line was implemented using the L78L33 linear
voltage regulator. However, the latter has a dropout voltage of 2V which
means that the L78L33 cannot output a stable +3.3V from a +5V input.

To solve the aforementioned problem the TC1017 LDO voltage regulator has
replaced the L78L33. The former has a low dropout voltage of 180mV (typ.) at
100mA load current.
Parts:
- C? (x16): footprint (none) -> Capacitors_SMD:C_1206_HandSoldering
- R? (x19): footprint (none) -> Resistors_SMD:R_1206_HandSoldering
- U? (x4): footprint (none) -> Housings_SOIC:SOIC-8_3.9x4.9mm_Pitch1.27mm
- U?: footprint (none) -> Housings_SSOP:TSSOP-14_4.4x5mm_Pitch0.65mm
- U?: footprint Package_TO_SOT_SMD:SOT-23 -> TO_SOT_Packages_SMD:SOT-23_Handsoldering
Other:
- moved on the sheet: C?, R?, U?

Commit message: [Signal Generator] Minor changes to output amplifier
1) The 2.2nF capacitor which created a real pole low-pass filter has
been removed. This is because its cutoff frequency was about 1.4MHz.
Whilst the generated function as a whole of the digital function
generator may be considered to have a frequency of 1MHz, the actual
frequency of the generated signal is in the tens of MHz (e.g.: 64MHz for
1MHz sine wave with 64 unique points).

2) The +2.5V voltage reference of the waveform amplification output stage has
been replaced by the AZ431-A. This is because the latter is much more
widespread and cheap when compared to the LM4040.
Parts:
- removed C?: 2.2nF, Capacitors_SMD:C_1206_HandSoldering, symbol Device:C
- removed C?: 100nF, Capacitors_SMD:C_1206_HandSoldering, symbol Device:C
- removed U?: LM4040CYM3-2.5-TR, TO_SOT_Packages_SMD:SOT-23_Handsoldering, symbol Reference_Voltage:LM4040DBZ-2.5
- added U?: AZ431AN-A, TO_SOT_Packages_SMD:SOT-23_Handsoldering, symbol ulib_Voltage_References:AZ431AN-A
Connections:
- wire segments 203 -> 198
Other:
- moved on the sheet: R?
Changed lines of the file:
@@
 Sheet 4 6
 Title "Digital Function Generator v2 - Output Circuitry"
-Date "2019-12-11"
+Date "2019-12-15"
 Rev "1"
 Comp "Petar Nikolov"
@@
 L Device:R R?
 U 1 1 5E0B7216
-P 5150 2800
-F 0 "R?" H 5220 2846 50  0000 L CNN
-F 1 "15R" H 5220 2755 50  0000 L CNN
-F 2 "Resistors_SMD:R_1206_HandSoldering" V 5080 2800 50  0001 C CNN
-F 3 "~" H 5150 2800 50  0001 C CNN
-	1    5150 2800
+P 5150 2550
+F 0 "R?" H 5220 2596 50  0000 L CNN
+F 1 "15R" H 5220 2505 50  0000 L CNN
+F 2 "Resistors_SMD:R_1206_HandSoldering" V 5080 2550 50  0001 C CNN
+F 3 "~" H 5150 2550 50  0001 C CNN
+	1    5150 2550
 	1    0    0    -1
 $EndComp
@@
 L Device:R R?
 U 1 1 5E0B72F3
-P 4650 2800
-F 0 "R?" H 4720 2846 50  0000 L CNN
-F 1 "15R" H 4720 2755 50  0000 L CNN
-F 2 "Resistors_SMD:R_1206_HandSoldering" V 4580 2800 50  0001 C CNN
-F 3 "~" H 4650 2800 50  0001 C CNN
-	1    4650 2800
-	1    0    0    -1
-$EndComp
-$Comp
-L Device:C C?
-U 1 1 5E0B73BA
-P 4900 2500
-F 0 "C?" V 4750 2500 50  0000 C CNN
-F 1 "2.2nF" V 5050 2500 50  0000 C CNN
-F 2 "Capacitors_SMD:C_1206_HandSoldering" H 4938 2350 50  0001 C CNN
-F 3 "~" H 4900 2500 50  0001 C CNN
-	1    4900 2500
-	0    1    1    0
-$EndComp
-Wire Wire Line
-	4650 2650 4650 2500
-Wire Wire Line
-	4650 2500 4750 2500
-Wire Wire Line
-	5050 2500 5150 2500
-Wire Wire Line
-	5150 2500 5150 2650
+P 4750 2550
+F 0 "R?" H 4820 2596 50  0000 L CNN
+F 1 "15R" H 4820 2505 50  0000 L CNN
+F 2 "Resistors_SMD:R_1206_HandSoldering" V 4680 2550 50  0001 C CNN
+F 3 "~" H 4750 2550 50  0001 C CNN
+	1    4750 2550
+	1    0    0    -1
+$EndComp
 $Comp
 L Device:R R?
 U 1 1 5E0D535D
-P 4650 3100
-F 0 "R?" H 4720 3146 50  0000 L CNN
-F 1 "10R" H 4720 3055 50  0000 L CNN
-F 2 "Resistors_SMD:R_1206_HandSoldering" V 4580 3100 50  0001 C CNN
-F 3 "~" H 4650 3100 50  0001 C CNN
-	1    4650 3100
+P 4750 2850
+F 0 "R?" H 4820 2896 50  0000 L CNN
+F 1 "10R" H 4820 2805 50  0000 L CNN
+F 2 "Resistors_SMD:R_1206_HandSoldering" V 4680 2850 50  0001 C CNN
+F 3 "~" H 4750 2850 50  0001 C CNN
+	1    4750 2850
 	1    0    0    -1
 $EndComp
@@
 L Device:R R?
 U 1 1 5E0D54AF
-P 5150 3100
-F 0 "R?" H 5220 3146 50  0000 L CNN
-F 1 "10R" H 5220 3055 50  0000 L CNN
-F 2 "Resistors_SMD:R_1206_HandSoldering" V 5080 3100 50  0001 C CNN
-F 3 "~" H 5150 3100 50  0001 C CNN
-	1    5150 3100
-	1    0    0    -1
-$EndComp
-Wire Wire Line
-	5150 3250 5150 3300
+P 5150 2850
+F 0 "R?" H 5220 2896 50  0000 L CNN
+F 1 "10R" H 5220 2805 50  0000 L CNN
+F 2 "Resistors_SMD:R_1206_HandSoldering" V 5080 2850 50  0001 C CNN
+F 3 "~" H 5150 2850 50  0001 C CNN
+	1    5150 2850
+	1    0    0    -1
+$EndComp
+Wire Wire Line
+	5150 3000 5150 3050
 $Comp
 L power:GNDA #PWR0208
 U 1 1 5E0DF805
-P 5150 3300
-F 0 "#PWR0208" H 5150 3050 50  0001 C CNN
-F 1 "GNDA" H 5155 3127 50  0000 C CNN
-F 2 "" H 5150 3300 50  0001 C CNN
-F 3 "" H 5150 3300 50  0001 C CNN
-	1    5150 3300
+P 5150 3050
+F 0 "#PWR0208" H 5150 2800 50  0001 C CNN
+F 1 "GNDA" H 5155 2877 50  0000 C CNN
+F 2 "" H 5150 3050 50  0001 C CNN
+F 3 "" H 5150 3050 50  0001 C CNN
+	1    5150 3050
 	1    0    0    -1
 $EndComp
@@
 L power:GNDA #PWR0209
 U 1 1 5E0DF869
-P 4650 3300
-F 0 "#PWR0209" H 4650 3050 50  0001 C CNN
-F 1 "GNDA" H 4655 3127 50  0000 C CNN
-F 2 "" H 4650 3300 50  0001 C CNN
-F 3 "" H 4650 3300 50  0001 C CNN
-	1    4650 3300
-	1    0    0    -1
-$EndComp
-Wire Wire Line
-	4650 3300 4650 3250
+P 4750 3050
+F 0 "#PWR0209" H 4750 2800 50  0001 C CNN
+F 1 "GNDA" H 4755 2877 50  0000 C CNN
+F 2 "" H 4750 3050 50  0001 C CNN
+F 3 "" H 4750 3050 50  0001 C CNN
+	1    4750 3050
+	1    0    0    -1
+$EndComp
+Wire Wire Line
+	4750 3050 4750 3000
 Wire Wire Line
 	5550 2300 5650 2300
-Wire Wire Line
-	5150 2500 5150 2100
-Connection ~ 5150 2500
-Wire Wire Line
-	4650 2300 4650 2500
-Connection ~ 4650 2500
 Text HLabel 4450 2100 0    50   Input ~ 0
 INA
@@
 	4150 750  7450 750
 Wire Wire Line
-	5250 2300 4650 2300
-$Comp
-L Reference_Voltage:LM4040DBZ-2.5 U?
-U 1 1 5E82D560
-P 1750 6800
-F 0 "U?" V 1750 6700 50  0000 R CNN
-F 1 "LM4040CYM3-2.5-TR" H 2150 6950 50  0000 R CNN
-F 2 "TO_SOT_Packages_SMD:SOT-23_Handsoldering" H 1750 6600 50  0001 C CIN
-F 3 "http://www.ti.com/lit/ds/symlink/lm4040-n.pdf" H 1750 6800 50  0001 C CIN
-	1    1750 6800
-	0    -1   -1   0
-$EndComp
+	5250 2300 4750 2300
 $Comp
 L power:GNDA #PWR0210
@@
 Wire Wire Line
 	1750 6550 1750 6600
-$Comp
-L Device:C C?
-U 1 1 5E82D57F
-P 1450 6800
-F 0 "C?" H 1200 6850 50  0000 L CNN
-F 1 "100nF" H 1100 6750 50  0000 L CNN
-F 2 "Capacitors_SMD:C_1206_HandSoldering" H 1488 6650 50  0001 C CNN
-F 3 "~" H 1450 6800 50  0001 C CNN
-	1    1450 6800
-	1    0    0    -1
-$EndComp
-$Comp
-L power:GNDA #PWR0212
-U 1 1 5E82D586
-P 1450 7000
-F 0 "#PWR0212" H 1450 6750 50  0001 C CNN
-F 1 "GNDA" H 1455 6827 50  0000 C CNN
-F 2 "" H 1450 7000 50  0001 C CNN
-F 3 "" H 1450 7000 50  0001 C CNN
-	1    1450 7000
-	1    0    0    -1
-$EndComp
-Wire Wire Line
-	1450 7000 1450 6950
-Wire Wire Line
-	1450 6600 1450 6650
-Wire Wire Line
-	1750 6600 1450 6600
 Wire Wire Line
 	1750 6600 2250 6600
@@
 	5150 2100 4450 2100
 Connection ~ 5150 2100
-Wire Wire Line
-	4650 2300 4450 2300
-Connection ~ 4650 2300
 Wire Notes Line
 	7450 750  7450 3550
@@
 Wire Wire Line
 	1350 3950 1550 3950
+Wire Wire Line
+	5150 2100 5150 2400
+Wire Wire Line
+	4750 2300 4750 2400
+Connection ~ 4750 2300
+Wire Wire Line
+	4450 2300 4750 2300
+$Comp
+L ulib_Voltage_References:AZ431AN-A U?
+U 1 1 5E172976
+P 1750 6800
+F 0 "U?" V 1796 6712 50  0000 R CNN
+F 1 "AZ431AN-A" V 1705 6712 50  0000 R CNN
+F 2 "TO_SOT_Packages_SMD:SOT-23_Handsoldering" H 1750 6800 50  0001 C CIN
+F 3 "https://www.diodes.com/assets/Datasheets/AZ431A.pdf" H 1750 6800 50  0001 C CIN
+	1    1750 6800
+	0    -1   -1   0
+$EndComp
+Wire Wire Line
+	1550 6800 1550 6600
+Wire Wire Line
+	1550 6600 1750 6600
 $EndSCHEMATC
